File: UrbanSteering.kicad_sch (KiCad schematic)
At the start: 21 parts

Commit message: PCB version 4
Parts:
- removed C?: 0.1 uF, symbol Device:C
- removed R?: 100, symbol Device:R
- removed R?: 68, symbol Device:R
- removed U?: Input (SR2), symbol 74xx:74HC595
- removed U?: Output (SR1), symbol 74xx:74HC595
- added C? (x3): 0.1uF, symbol pspice:C
- added J? (x4): Conn_01x02_Female, symbol Connector:Conn_01x02_Female
- added R? (x6): 68, symbol Device:R
- added R? (x7): 10k, symbol Device:R
- added U?: 74HC595PW, SOT403-1_NXP, symbol 2022-11-01_22-08-37:74HC595PW
- added U?: 74HC597D, SOT109-1_NEX, symbol 2022-11-01_22-13-43:74HC597D
- J4: value (none) -> STM32L432; footprint (none) -> schematic:STM32L432
- S1: value (none) -> HORN; footprint (none) -> LP11EE1NCSYG:LP11OA1TCSYY
- S2: value (none) -> INDICATORS; footprint (none) -> M2013TXG13DA:M2013TXG13DA
- S3: value (none) -> IGNITION; footprint (none) -> LP11EE1NCSYG:LP11EE1NCSYG
- S4: value (none) -> WIPERS; footprint (none) -> LP11EE1NCSYG:LP11EE1NCSYG
- S5: value (none) -> LIGHTS; footprint (none) -> LP11EE1NCSYG:LP11EE1NCSYG
- TP2: value (none) -> HAZARDS; footprint (none) -> LP11EE1NCSYG:LP11EE1NCSYG
- U1: value (none) -> MCP2562; footprint (none) -> footprints:MCP2562FD-H&slash_P
Connections:
- net +3V3 is gone; now on net VCC: S1.1, S3.1, TP2.1
- net GND: now also J?.1 (Pin_1), J?.2 (Pin_2), J?.2 (Pin_2), J?.3 (Pin_3), J?.7 (Pin_7), U1.2 (VSS), U1.8 (STBY), C?.2, C?.2, C?.2, J?.2 (Pin_2), J?.2 (Pin_2), J?.2 (Pin_2), R?.1, R?.1, R?.1, R?.1, R?.1, R?.1, R?.1, U?.13 (OE*), U?.13 (PL*), U?.8 (GND), U?.8 (GND)
- net HAZARDS: now also R?.2, U?.7 (D7)
- net HORN: now also R?.2, U?.5 (D5)
- net IGNITION: now also R?.2, U?.6 (D6)
- net Latch: now also U?.12 (STCP), U?.12 (ST_CP)
- net SR2-STM: now also U?.9 (Q)
- net SRCLK: now also U?.11 (SHCP), U?.11 (SH_CP)
- net STM-SR1: now also U?.14 (DS)
- net VCC: now also J?.1 (Pin_1), J?.2 (Pin_2), J?.4 (Pin_4), J?.6 (Pin_6), J?.8 (Pin_8), S1.LC, S2.2 (COM), S3.LC, S4.1, S4.LC, S5.1, S5.LC, TP2.LC, U1.5 (VIO), C?.1, C?.1, J?.1 (Pin_1), U?.10 (MR*), U?.10 (MR*), U?.16 (VCC), U?.16 (VCC)
- net at S3.L1 (L1_Y): now also R?.2
- net at S3.L2 (L2_G): now also R?.2
- net WIPRES: now reaches S4.2
- net WIPRES: now also R?.2, U?.3 (D3)
- net at S4.L2 (L2_G): now also R?.1
- net LIGHTS: now reaches S5.2
- net LIGHTS: now also R?.2, U?.4 (D4)
- net at S5.L2 (L2_G): now also R?.1
- net at TP2.L1 (L1_Y): now also R?.2
- net at S1.L1 (L1_Y): now also R?.2
- net IND_LEFT: now reaches S2.LEFT
- net IND_LEFT: now also R?.2, U?.2 (D2)
- net IND_RIGHT: now reaches S2.RIGHT
- net IND_RIGHT: now also R?.2, U?.1 (D1)
- net +5V: now reaches U1.3 (VDD)
- net +5V: now also J4.27 (5V), C?.1, J?.1 (Pin_1)
- net RXD: now reaches U1.4 (RXD)
- net RXD: now also J4.13 (D10)
- net CANL: now reaches U1.6 (CANL)
- net CANL: now also J?.5 (Pin_5), R?.2, J?.1 (Pin_1)
- net CANH: now reaches U1.7 (CANH)
- net CANH: now also J?.2 (Pin_2), J?.4 (Pin_4), J?.2 (Pin_2)
- net LCD_DC: now reaches J4.10 (D7)
- net LCD_DC: now also J?.5 (Pin_5)
- net LCD_CS: now reaches J4.12 (D9)
- net LCD_CS: now also J?.3 (Pin_3)
- net LCD_MOSI: now reaches J4.14 (D11)
- net LCD_MOSI: now also J?.2 (Pin_2), J?.6 (Pin_6)
- net LCD_MISO: now reaches J4.15 (D12)
- net LCD_MISO: now also J?.3 (Pin_3), J?.9 (Pin_9)
- net LCD_SCK: now reaches J4.16 (D13)
- net LCD_SCK: now also J?.4 (Pin_4), J?.7 (Pin_7)
- net SD_CS: now reaches J4.19 (A0)
- net SD_CS: now also J?.1 (Pin_1)
- net ProximInput: now reaches J4.20 (A1)
- net ProximInput: now also J?.3 (Pin_3)
- net JoystickY: now reaches J4.21 (A2)
- net JoystickY: now also J?.4 (Pin_4)
- net JoystickX: now reaches J4.22 (A3)
- net JoystickX: now also J?.3 (Pin_3)
- net Throttle: now reaches J4.25 (A6)
- net Throttle: now also J?.2 (Pin_2)
- net +12V: now reaches J4.30 (VIN)
- net +12V: now also J?.8 (Pin_8), J?.1 (Pin_1)
- net at J?.1 (Pin_1): now also R?.1
- net SW_JOY: now reaches J?.5 (Pin_5)
- net SW_JOY: now also U?.15 (D0)
- new net HAZARDS_OFF: R?.1
- new net HAZARDS_ON: U?.6 (Q6)
- new net HORN_PRESSED: R?.1, U?.4 (Q4)
- new net IGNITION_OFF: R?.1
- new net IGNITION_ON: R?.1, U?.5 (Q5)
- new net LIGHTS_OFF: U?.3 (Q3)
- new net LIGHTS_ON: R?.2, U?.2 (Q2)
- new net WIPRES_ON: R?.2, U?.1 (Q1)
- no-connect marks 17 -> 19
Other:
- moved on the sheet: J4, J?, R?, S1, S2, S3, S4, S5, TP2, U1

Commit message: PCB version-4 with mounting holes
Parts:
- removed J? (x3): Conn_01x02_Female, symbol Connector:Conn_01x02_Female
- added H1, H2, H3, H4: MountingHole, symbol Mechanical:MountingHole
- added J10, J11, J12, J13, J8: Conn_01x01_Female, symbol Connector:Conn_01x01_Female
- added R5: 10k, symbol Device:R
- gave numbers to parts that had none: 27
Connections:
- net HAZARDS_ON is gone; now on net LED_HAZARDS_ON: U2.6 (Q6)
- net LIGHTS_OFF is gone; now on net LED_HORN_PRESSED: U2.3 (Q3)
- net +12V: now also J11.1 (Pin_1)
- net +5V: now also J12.1 (Pin_1)
- net GND: now also J13.1 (Pin_1)
- net LCD_DC: now also J4.23 (A4); no longer J4.10 (D7)
- net ProximInput: now also J8.1 (Pin_1)
- net SW_JOY: now also R5.1
- net VCC: now also J10.1 (Pin_1), R5.2
- net HAZARDS renamed BTN_HAZARDS
- net HAZARDS_OFF renamed LED_HAZARDS_ON
- net HORN renamed BTN_HORN
- net HORN_PRESSED renamed LED_HORN_PRESSED
- net LED_HORN_PRESSED: no longer U2.4 (Q4)
- net IGNITION renamed BTN_IGNITION
- net IGNITION_OFF renamed LED_IGNITION_OFF
- net LED_IGNITION_OFF: now also U2.4 (Q4)
- net IGNITION_ON renamed LED_IGNITION_ON
- net IND_LEFT renamed BTN_IND_LEFT
- net IND_RIGHT renamed BTN_IND_RIGHT
- net LIGHTS renamed BTN_LIGHTS
- net LIGHTS_ON renamed LED_LIGHTS_ON
- net WIPRES renamed BTN_WIPERS
- net WIPRES_ON renamed LED_WIPERS_ON
- no-connect marks 19 -> 20
Other:
- moved on the sheet: C1, C3, J5, J6, J7, R2, R3, R4, U2, U3

Commit message: started pcb layout
Parts:
- added H5, H6: MountingHole, MountingHole:MountingHole_3.2mm_M3, symbol Mechanical:MountingHole
- C1, C2, C3: footprint (none) -> Capacitor_SMD:C_0805_2012Metric
- H1, H2, H3, H4: footprint (none) -> MountingHole:MountingHole_3.2mm_M3
- J1: footprint (none) -> Connector_PinHeader_2.54mm:PinHeader_1x05_P2.54mm_Vertical
- J10, J11, J12, J13, J8: footprint (none) -> Connector_PinHeader_2.54mm:PinHeader_1x01_P2.54mm_Vertical
- J2: footprint (none) -> KiCad:705510007
- J3, J7: footprint (none) -> Connector_PinHeader_2.54mm:PinHeader_1x02_P2.54mm_Vertical
- J5: footprint (none) -> Connector_PinHeader_2.54mm:PinHeader_1x14_P2.54mm_Vertical
- J6: footprint (none) -> Connector_PinHeader_2.54mm:PinHeader_1x04_P2.54mm_Vertical
- J9: footprint (none) -> Supermileage_PCB:705510003
- R1, R10, R11, R12, R13, R14, R15, R16, R2, R3, R4, R5, R6, R7, R8, R9: footprint (none) -> Resistor_SMD:R_0805_2012Metric
- U2: footprint SOT403-1_NXP -> Package_SO:TSSOP-16-1EP_4.4x5mm_P0.65mm
- U3: footprint SOT109-1_NEX -> Package_SO:TSSOP-16-1EP_4.4x5mm_P0.65mm
Connections:
- net GND: now also S2.SH1 (SH), S2.SH2 (SH), S2.SH3 (SH), S2.SH4 (SH)
- no-connect marks 20 -> 19

Commit message: adjusts position of some footprints, adds most required labels, deletes existing traces, flips LCD orientation, and adjusts netclass sizes
Parts:
- H1, H2, H3, H4, H5, H6: value MountingHole -> M3
- J2: footprint KiCad:705510007 -> Connector_Molex:705510007
- J5: value Screen_left -> Screen_Left
- J6: value Screen_right -> Screen_Right
- J9: footprint Supermileage_PCB:705510003 -> Connector_Molex:705510003
- TP1: renamed from J7; value Conn_01x02_Female -> CAN
- TP2: renamed from J8; value Conn_01x01_Female -> Proxim
- TP3: renamed from J10; value Conn_01x01_Female -> 3v3
- TP4: renamed from J11; value Conn_01x01_Female -> 12v
- TP5: renamed from J12; value Conn_01x01_Female -> 5v
- TP6: renamed from J13; value Conn_01x01_Female -> GND
- renumbered TP2 to S6
Connections:
- net GND: now also J1.5 (Pin_5); no longer J1.1 (Pin_1)
- net JoystickY: now also J1.2 (Pin_2); no longer J1.4 (Pin_4)
- net SW_JOY: now also J1.1 (Pin_1), R5.2; no longer J1.5 (Pin_5), R5.1
- net VCC: now also J1.4 (Pin_4), R5.1; no longer J1.2 (Pin_2), R5.2
Other:
- moved on the sheet: R5

Commit message: added fuse to schematic - layout to be changed
Parts:
- added F1: Fuse, Fuse:Fuse_1206_3216Metric, symbol Device:Fuse
Connections:
- net +12V: now also F1.2; no longer J2.8 (Pin_8)
- net CANH: now also J2.5 (Pin_5); no longer J2.4 (Pin_4)
- net CANL: now also J2.3 (Pin_3); no longer J2.5 (Pin_5)
- net GND: now also J2.4 (Pin_4); no longer J2.3 (Pin_3)
- new net: F1.1, J2.8 (Pin_8)
Changed lines of the file:
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@@
     (company "UBC SUPERMILEAGE")
   )
+  (junction (at 68.58 30.48) (diameter 0) (color 0 0 0 0)
+  )
   (junction (at 95.25 152.4) (diameter 0) (color 0 0 0 0)
   )
   (junction (at 271.78 60.96) (diameter 0) (color 0 0 0 0)
-  )
-  (junction (at 63.5 25.4) (diameter 0) (color 0 0 0 0)
   )
   (junction (at 20.32 60.96) (diameter 0) (color 0 0 0 0)
@@
     (stroke (width 0) (type default) (color 0 0 0 0))
   )
+  (wire (pts (xy 81.28 43.18) (xy 81.28 29.21))
+    (stroke (width 0) (type default) (color 0 0 0 0))
+  )
   (wire (pts (xy 113.03 102.87) (xy 99.06 102.87))
     (stroke (width 0) (type default) (color 0 0 0 0))
@@
     (stroke (width 0) (type default) (color 0 0 0 0))
   )
+  (wire (pts (xy 63.5 30.48) (xy 63.5 33.02))
+    (stroke (width 0) (type default) (color 0 0 0 0))
+  )
   (wire (pts (xy 252.73 80.01) (xy 251.46 80.01))
     (stroke (width 0) (type default) (color 0 0 0 0))
@@
     (stroke (width 0) (type default) (color 0 0 0 0))
   )
-  (wire (pts (xy 78.74 29.21) (xy 78.74 34.29))
+  (wire (pts (xy 78.74 29.21) (xy 78.74 31.75))
     (stroke (width 0) (type default) (color 0 0 0 0))
   )
@@
     (stroke (width 0) (type default) (color 0 0 0 0))
   )
-  (wire (pts (xy 63.5 25.4) (xy 63.5 33.02))
-    (stroke (width 0) (type default) (color 0 0 0 0))
-  )
   (wire (pts (xy 189.23 148.59) (xy 180.34 148.59))
     (stroke (width 0) (type default) (color 0 0 0 0))
@@
     (stroke (width 0) (type default) (color 0 0 0 0))
   )
-  (wire (pts (xy 68.58 29.21) (xy 68.58 33.02))
+  (wire (pts (xy 68.58 29.21) (xy 68.58 30.48))
     (stroke (width 0) (type default) (color 0 0 0 0))
   )
@@
     (stroke (width 0) (type default) (color 0 0 0 0))
   )
-  (wire (pts (xy 81.28 29.21) (xy 81.28 39.37))
+  (wire (pts (xy 68.58 30.48) (xy 68.58 33.02))
     (stroke (width 0) (type default) (color 0 0 0 0))
   )
@@
     (stroke (width 0) (type default) (color 0 0 0 0))
   )
-  (wire (pts (xy 63.5 21.59) (xy 63.5 25.4))
+  (wire (pts (xy 63.5 21.59) (xy 63.5 22.86))
     (stroke (width 0) (type default) (color 0 0 0 0))
   )
@@
   )
   (wire (pts (xy 106.68 92.71) (xy 104.14 92.71))
+    (stroke (width 0) (type default) (color 0 0 0 0))
+  )
+  (wire (pts (xy 67.31 30.48) (xy 68.58 30.48))
     (stroke (width 0) (type default) (color 0 0 0 0))
   )
@@
     (effects (font (size 1.27 1.27)) (justify left bottom))
   )
-  (label "CANH" (at 78.74 34.29 90)
-    (effects (font (size 1.27 1.27)) (justify left bottom))
-  )
   (label "CANH" (at 209.55 20.32 0)
     (effects (font (size 1.27 1.27)) (justify left bottom))
@@
     (effects (font (size 1.27 1.27)) (justify left bottom))
   )
+  (label "CANL" (at 81.28 43.18 90)
+    (effects (font (size 1.27 1.27)) (justify left bottom))
+  )
   (label "BTN_IND_LEFT" (at 26.67 82.55 0)
-    (effects (font (size 1.27 1.27)) (justify left bottom))
-  )
-  (label "CANL" (at 76.2 34.29 90)
     (effects (font (size 1.27 1.27)) (justify left bottom))
   )
@@
   (label "LCD_MISO" (at 186.69 46.99 180)
     (effects (font (size 1.27 1.27)) (justify right bottom))
+  )
+  (label "CANH" (at 76.2 34.29 90)
+    (effects (font (size 1.27 1.27)) (justify left bottom))
   )
   (symbol (lib_id "LP11EE1NCSYG:LP11EE1NCSYG") (at 243.84 106.68 0) (mirror y) (unit 1)
@@
     (pin "9")
   )
+  (symbol (lib_id "Device:Fuse") (at 63.5 26.67 180) (unit 1)
+    (in_bom yes) (on_board yes)
+    (property "Reference" "F1" (id 0) (at 59.69 25.4 0)
+      (effects (font (size 1.27 1.27)) (justify right))
+    )
+    (property "Value" "Fuse" (id 1) (at 57.15 26.67 0)
+      (effects (font (size 1.27 1.27)) (justify right))
+    )
+    (property "Footprint" "Fuse:Fuse_1206_3216Metric" (id 2) (at 65.278 26.67 90)
+      (effects (font (size 1.27 1.27)) hide)
+    )
+    (property "Datasheet" "~" (id 3) (at 63.5 26.67 0)
+      (effects (font (size 1.27 1.27)) hide)
+    )
+    (pin "1")
+    (pin "2")
+  )
   (symbol (lib_id "Device:R") (at 231.14 80.01 90) (unit 1)
     (in_bom yes) (on_board yes)
@@
     (pin "1")
   )
-  (symbol (lib_id "power:PWR_FLAG") (at 63.5 25.4 90) (unit 1)
-    (in_bom yes) (on_board yes) (fields_autoplaced)
-    (property "Reference" "#FLG0102" (id 0) (at 61.595 25.4 0)
-      (effects (font (size 1.27 1.27)) hide)
-    )
-    (property "Value" "PWR_FLAG" (id 1) (at 59.69 25.3999 90)
-      (effects (font (size 1.27 1.27)) (justify left))
-    )
-    (property "Footprint" "" (id 2) (at 63.5 25.4 0)
-      (effects (font (size 1.27 1.27)) hide)
-    )
-    (property "Datasheet" "~" (id 3) (at 63.5 25.4 0)
+  (symbol (lib_id "power:PWR_FLAG") (at 67.31 30.48 90) (unit 1)
+    (in_bom yes) (on_board yes)
+    (property "Reference" "#FLG0102" (id 0) (at 65.405 30.48 0)
+      (effects (font (size 1.27 1.27)) hide)
+    )
+    (property "Value" "PWR_FLAG" (id 1) (at 62.23 30.48 90)
+      (effects (font (size 1.27 1.27)) (justify left))
+    )
+    (property "Footprint" "" (id 2) (at 67.31 30.48 0)
+      (effects (font (size 1.27 1.27)) hide)
+    )
+    (property "Datasheet" "~" (id 3) (at 67.31 30.48 0)
       (effects (font (size 1.27 1.27)) hide)
     )
@@
     (pin "1")
   )
-  (symbol (lib_id "power:GND") (at 81.28 39.37 0) (unit 1)
-    (in_bom yes) (on_board yes)
-    (property "Reference" "#PWR015" (id 0) (at 81.28 45.72 0)
-      (effects (font (size 1.27 1.27)) hide)
-    )
-    (property "Value" "GND" (id 1) (at 78.74 43.18 0)
-      (effects (font (size 1.27 1.27)) (justify left))
-    )
-    (property "Footprint" "" (id 2) (at 81.28 39.37 0)
-      (effects (font (size 1.27 1.27)) hide)
-    )
-    (property "Datasheet" "" (id 3) (at 81.28 39.37 0)
+  (symbol (lib_id "power:GND") (at 78.74 31.75 0) (unit 1)
+    (in_bom yes) (on_board yes)
+    (property "Reference" "#PWR015" (id 0) (at 78.74 38.1 0)
+      (effects (font (size 1.27 1.27)) hide)
+    )
+    (property "Value" "GND" (id 1) (at 76.2 35.56 0)
+      (effects (font (size 1.27 1.27)) (justify left))
+    )
+    (property "Footprint" "" (id 2) (at 78.74 31.75 0)
+      (effects (font (size 1.27 1.27)) hide)
+    )
+    (property "Datasheet" "" (id 3) (at 78.74 31.75 0)
       (effects (font (size 1.27 1.27)) hide)
     )
@@
       (reference "C3") (unit 1) (value "0.1uF") (footprint "Capacitor_SMD:C_0805_2012Metric")
     )
+    (path "/35420b5d-695b-4fd4-8e5c-6f7cbfc14aa6"
+      (reference "F1") (unit 1) (value "Fuse") (footprint "Fuse:Fuse_1206_3216Metric")
+    )
     (path "/1a4edfad-ad16-4700-8a23-d86dc27a3159"

Commit message: added labels
Parts:
- S3: value IGNITION -> RUN/STOP
Changed lines of the file:
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@@
     (in_bom yes) (on_board yes)
     (property "Reference" "S3" (id 0) (at 240.03 96.52 0))
-    (property "Value" "IGNITION" (id 1) (at 247.65 96.52 0))
+    (property "Value" "RUN/STOP" (id 1) (at 247.65 96.52 0))
     (property "Footprint" "LP11EE1NCSYG:LP11EE1NCSYG" (id 2) (at 243.84 118.11 0)
       (effects (font (size 1.27 1.27)) hide)
@@
     )
     (path "/00000000-0000-0000-0000-00005f9e641c"
-      (reference "S3") (unit 1) (value "IGNITION") (footprint "LP11EE1NCSYG:LP11EE1NCSYG")
+      (reference "S3") (unit 1) (value "RUN/STOP") (footprint "LP11EE1NCSYG:LP11EE1NCSYG")
     )
     (path "/00000000-0000-0000-0000-00005f9fb1ed"

Commit message: Physical hardware changes replicated in KiCad design
Parts:
- added R17: 10k, Resistor_SMD:R_0805_2012Metric, symbol Device:R
Connections:
- net GND: now also R17.2; no longer U3.13 (PL*)
- net Latch: now also U3.13 (PL*)
- net ProximInput: now also R17.1
Changed lines of the file:
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@@
   (junction (at 189.23 130.81) (diameter 0) (color 0 0 0 0)
+  )
+  (junction (at 180.34 140.97) (diameter 0) (color 0 0 0 0)
   )
   (junction (at 278.13 60.96) (diameter 0) (color 0 0 0 0)
@@
     (stroke (width 0) (type default) (color 0 0 0 0))
   )
+  (wire (pts (xy 205.74 27.94) (xy 205.74 29.21))
+    (stroke (width 0) (type default) (color 0 0 0 0))
+  )
   (wire (pts (xy 31.75 22.86) (xy 31.75 26.67))
     (stroke (width 0) (type default) (color 0 0 0 0))
@@
     (stroke (width 0) (type default) (color 0 0 0 0))
   )
+  (wire (pts (xy 205.74 38.1) (xy 205.74 36.83))
+    (stroke (width 0) (type default) (color 0 0 0 0))
+  )
   (wire (pts (xy 81.28 43.18) (xy 81.28 29.21))
     (stroke (width 0) (type default) (color 0 0 0 0))
@@
     (stroke (width 0) (type default) (color 0 0 0 0))
   )
+  (wire (pts (xy 180.34 138.43) (xy 180.34 140.97))
+    (stroke (width 0) (type default) (color 0 0 0 0))
+  )
   (wire (pts (xy 25.4 96.52) (xy 25.4 99.06))
     (stroke (width 0) (type default) (color 0 0 0 0))
@@
   )
   (wire (pts (xy 251.46 39.37) (xy 256.54 39.37))
-    (stroke (width 0) (type default) (color 0 0 0 0))
-  )
-  (wire (pts (xy 180.34 138.43) (xy 193.04 138.43))
     (stroke (width 0) (type default) (color 0 0 0 0))
   )
@@
     (pin "1")
   )
+  (symbol (lib_id "Device:R") (at 205.74 33.02 0) (unit 1)
+    (in_bom yes) (on_board yes) (fields_autoplaced)
+    (property "Reference" "R17" (id 0) (at 208.28 31.7499 0)
+      (effects (font (size 1.27 1.27)) (justify left))
+    )
+    (property "Value" "10k" (id 1) (at 208.28 34.2899 0)
+      (effects (font (size 1.27 1.27)) (justify left))
+    )
+    (property "Footprint" "Resistor_SMD:R_0805_2012Metric" (id 2) (at 203.962 33.02 90)
+      (effects (font (size 1.27 1.27)) hide)
+    )
+    (property "Datasheet" "~" (id 3) (at 205.74 33.02 0)
+      (effects (font (size 1.27 1.27)) hide)
+    )
+    (pin "1")
+    (pin "2")
+  )
   (symbol (lib_id "power:+5V") (at 99.06 95.25 0) (unit 1)
     (in_bom yes) (on_board yes)
@@
     (pin "1")
   )
-  (symbol (lib_id "power:GND") (at 193.04 138.43 0) (unit 1)
-    (in_bom yes) (on_board yes)
-    (property "Reference" "#PWR036" (id 0) (at 193.04 144.78 0)
-      (effects (font (size 1.27 1.27)) hide)
-    )
-    (property "Value" "GND" (id 1) (at 191.77 142.24 0)
-      (effects (font (size 1.27 1.27)) (justify left))
-    )
-    (property "Footprint" "" (id 2) (at 193.04 138.43 0)
-      (effects (font (size 1.27 1.27)) hide)
-    )
-    (property "Datasheet" "" (id 3) (at 193.04 138.43 0)
-      (effects (font (size 1.27 1.27)) hide)
-    )
-    (pin "1")
-  )
   (symbol (lib_id "Mechanical:MountingHole") (at 142.24 175.26 0) (unit 1)
     (in_bom yes) (on_board yes)
@@
     (pin "1")
   )
+  (symbol (lib_id "power:GND") (at 205.74 38.1 0) (unit 1)
+    (in_bom yes) (on_board yes) (fields_autoplaced)
+    (property "Reference" "#PWR0102" (id 0) (at 205.74 44.45 0)
+      (effects (font (size 1.27 1.27)) hide)
+    )
+    (property "Value" "GND" (id 1) (at 205.74 43.18 0))
+    (property "Footprint" "" (id 2) (at 205.74 38.1 0)
+      (effects (font (size 1.27 1.27)) hide)
+    )
+    (property "Datasheet" "" (id 3) (at 205.74 38.1 0)
+      (effects (font (size 1.27 1.27)) hide)
+    )
+    (pin "1")
+  )
   (symbol (lib_id "power:GND") (at 134.62 86.36 0) (unit 1)
     (in_bom yes) (on_board yes)
@@
       (reference "#PWR035") (unit 1) (value "VCC") (footprint "")
     )
-    (path "/64bf41ab-4318-41e5-8d1c-92f19293a031"
-      (reference "#PWR036") (unit 1) (value "GND") (footprint "")
-    )
     (path "/f812c6df-3df8-4f7e-ba62-1410fa3e9769"
       (reference "#PWR037") (unit 1) (value "GND") (footprint "")
@@
       (reference "#PWR0101") (unit 1) (value "GND") (footprint "")
     )
+    (path "/e34a7e38-f492-4606-8210-332093323ddc"
+      (reference "#PWR0102") (unit 1) (value "GND") (footprint "")
+    )
     (path "/8d2a535a-5176-4060-b46d-a5d0336c5a91"
       (reference "C1") (unit 1) (value "0.1uF") (footprint "Capacitor_SMD:C_0805_2012Metric")
@@
       (reference "R16") (unit 1) (value "10k") (footprint "Resistor_SMD:R_0805_2012Metric")
     )
+    (path "/06e01605-302b-49f0-bda7-d98c199be604"
+      (reference "R17") (unit 1) (value "10k") (footprint "Resistor_SMD:R_0805_2012Metric")
+    )
     (path "/00000000-0000-0000-0000-00005fa78095"
